File: hardware/esp32_clones/esp32_clones.kicad_pcb (KiCad board)
At the start: 2 copper layers, 110 x 60 mm, 27 parts, among them J2 USB_A, J3 USB_A, J4 USB_A, J5 Micro_SD_Card, J6 Barrel_Jack, J7 DA15_Pins, J9 AudioJack2_Ground

Commit message: Refactor code structure for improved readability and maintainability
Parts:
- removed C2: C, Capacitor_SMD:C_0805_2012Metric_Pad1.18x1.45mm_HandSolder
- removed R10: 1k, Resistor_SMD:R_0805_2012Metric_Pad1.20x1.40mm_HandSolder
- removed kibuzzard-6A32A222: G***, kibuzzard-6A32A222
- removed kibuzzard-6A32A22E: G***, kibuzzard-6A32A22E
- added C3: 10UF, Capacitor_SMD:CP_Elec_6.3x3, F.Cu at (133.2, 79.7)
- added C4: 100NF, Capacitor_SMD:C_0805_2012Metric_Pad1.18x1.45mm_HandSolder, F.Cu at (168.8, 84.1)
- added C5: 47NF, Capacitor_SMD:C_0805_2012Metric_Pad1.18x1.45mm_HandSolder, F.Cu at (172.3, 84.2)
- added C6: 47NF, Capacitor_SMD:C_0805_2012Metric_Pad1.18x1.45mm_HandSolder, F.Cu at (131.7, 91.7)
- added C7: 100NF, Capacitor_SMD:C_0805_2012Metric_Pad1.18x1.45mm_HandSolder, F.Cu at (125.6, 91.7)
- added C8: 10UF, Capacitor_SMD:CP_Elec_6.3x3, F.Cu at (121.7, 79.7)
- added R11: 330KR, Resistor_SMD:R_0805_2012Metric_Pad1.20x1.40mm_HandSolder, F.Cu at (175.6, 84.2)
- added R12: 300KR, Resistor_SMD:R_0805_2012Metric_Pad1.20x1.40mm_HandSolder, F.Cu at (184.2, 83.2)
- added R13: 300KR, Resistor_SMD:R_0805_2012Metric_Pad1.20x1.40mm_HandSolder, F.Cu at (180.9, 83.3)
- added R14: 330KR, Resistor_SMD:R_0805_2012Metric_Pad1.20x1.40mm_HandSolder, F.Cu at (137.7, 91.7)
- moved kibuzzard-6A32A25A 67.1 mm to (167.8, 35.0)
- moved G*** 66.7 mm to (168.0, 28.2)
- moved J9 14.4 mm to (127.7, 67.0)
- moved U1 0.06 mm to (171.5, 89.4)
Connections:
- J9 pad S: Net-(C2-Pad1) -> Net-(C3-Pad2)
- J9 pad T: Net-(C2-Pad1) -> Net-(C8-Pad2)
- U1 pad 7: unconnected-(U1-IO48-Pad7) -> Net-(U1-IO48)
Routing:
- net Net-(C6-Pad2): track 0.00 -> 54.3 mm, vias 0 -> 2
- net Net-(C7-Pad2): track 0.00 -> 26.6 mm, vias 0 -> 2
- net Net-(C2-Pad1): track 25.7 -> 0.00 mm
- net Net-(U1-IO47): track 29.5 -> 5.58 mm
- net Net-(C8-Pad2): track 0.00 -> 23.4 mm
- net Net-(C3-Pad2): track 0.00 -> 22.7 mm
- net Net-(U1-IO48): track 0.00 -> 5.94 mm
- net Net-(C5-Pad1): track 0.00 -> 5.40 mm
- net Net-(J5-CLK): track 70.0 -> 72.5 mm
- net Net-(J5-DAT0): track 65.5 -> 67.1 mm
- net Net-(J5-CMD): track 73.9 -> 73.2 mm
