File: hardware/esp32_clones/esp32_clones.kicad_sch (KiCad schematic)
At the start: 31 parts, among them J2 USB_A, J3 USB_A, J4 USB_A, J5 Micro_SD_Card, J6 Barrel_Jack, J7 DA15_Pins, J9 AudioJack2_Ground

Commit message: Add production files for ESP32 clones including BOM, designators, netlist, and positions
- Created bom.csv to define components and their specifications.
- Added designators.csv to map designators to their respective values.
- Introduced netlist.ipc for electrical connections and layout.
- Added positions.csv to specify component placements on the PCB.
Parts:
- R1: renamed from R7; value 10KR -> 10K
- R10: renamed from R3; value 1.2KR -> 1.2K
- R11: renamed from R4; value 560R -> 560
- R12: renamed from R2; value 1.2KR -> 1.2K
- R13: renamed from R1; value 560R -> 560
- R2: renamed from R11; value 330KR -> 330
- R3: renamed from R14; value 330KR -> 330
- R4: renamed from R8; value 10KR -> 10K
- R5: renamed from R12; value 300KR -> 330
- R6: renamed from R13; value 300KR -> 330
- R7: renamed from R9; value 10KR -> 10K
- R8: renamed from R5; value 1.2KR -> 1.2K
- R9: renamed from R6; value 560R -> 560
- renumbered C3 to C2, C8 to C3, C7 to C5, C5 to C6, C6 to C7, J6 to J1, J5 to J2, J9 to J3, J1 to J4, J8 to J5, J2 to J6, J3 to J7, J4 to J8, J7 to J9
Connections:
- net GND: now also J5.3; no longer J5.2
- net at J5.1: no longer U1.25 (RST)
- new net: J5.2, U1.25 (RST)
Other:
- moved on the sheet: C3, C5, C7, J3, R3, R6
